File: modulo_puente_h/modulo_puente_h.kicad_pcb (KiCad board)
At the start: 2 copper layers, 63 x 50 mm, 16 parts, among them J1 Conn_01x07_Pin, M1 Motor_IZQ, M2 Motor_DER, U1 L298N

Commit message: fix: Las pistas van del lado de las soldaduras
No se puede soldar en el plástico :/
Parts:
- R1, R2: moved to B.Cu
- moved R1 0.50 mm to (53.0, 79.5)
Routing:
- net GND: track 67.9 -> 53.3 mm
- net Net-(U1-SENSE_A): track 21.9 -> 14.3 mm
- net Net-(U1-SENSE_B): track 14.9 -> 12.8 mm
- added copper zone on B.Cu, net GND
- removed copper zone on F.Cu, net GND
